File: main_board/main_board.sch (KiCad schematic (older format))
At the start: 55 parts

Commit message: Finalize schematic
Parts:
- added Q10, Q19, Q20, Q9: 2N7002P, Package_TO_SOT_SMD:SOT-23_Handsoldering, symbol Device:Q_NMOS_GSD
- added R10, R14, R16, R17, R21, R6, R8: 50, Resistor_SMD:R_0201_0603Metric_Pad0.64x0.40mm_HandSolder, symbol Device:R_Small
- added R11, R12, R19, R20: 1k, Resistor_SMD:R_0201_0603Metric_Pad0.64x0.40mm_HandSolder, symbol Device:R_Small
- added TP2: 3v3, TestPoint:TestPoint_Pad_D1.5mm, symbol Connector:TestPoint
- C1, C3: renamed from C?; footprint (none) -> Capacitor_SMD:C_1206_3216Metric
- C2, C6: renamed from C?; footprint (none) -> Capacitor_SMD:C_0603_1608Metric_Pad1.08x0.95mm_HandSolder
- C4, C5: renamed from C?; value 22u -> 22u 5v; footprint (none) -> Capacitor_SMD:C_0603_1608Metric_Pad1.08x0.95mm_HandSolder
- C7, C8: renamed from C?; value 22u -> 22u 7v; footprint (none) -> Capacitor_SMD:C_0805_2012Metric_Pad1.18x1.45mm_HandSolder
- D1: renamed from D?; footprint (none) -> good_things:smd_diode_sod_106
- J1: renamed from J?; footprint (none) -> TerminalBlock_Phoenix:TerminalBlock_Phoenix_MKDS-1,5-2_1x02_P5.00mm_Horizontal
- J2: renamed from J?; footprint (none) -> Connector_PinHeader_2.54mm:PinHeader_1x03_P2.54mm_Vertical
- J3: renamed from J?; footprint (none) -> TerminalBlock_Phoenix:TerminalBlock_Phoenix_MKDS-1,5-3_1x03_P5.00mm_Horizontal
- J4, J5: renamed from J?; footprint (none) -> Connector_RJ:RJ45_BEL_SS74301-00x_Vertical
- J6, J7: renamed from J?; footprint (none) -> Connector_PinHeader_2.54mm:PinHeader_1x07_P2.54mm_Vertical
- L1, L2: renamed from L?; footprint (none) -> good_things:smd_inductor_0806_2016metric
- Q1, Q12, Q15, Q18, Q24, Q3, Q7: renamed from Q?; footprint (none) -> Package_TO_SOT_SMD:SOT-323_SC-70_Handsoldering
- Q11, Q13, Q14, Q16, Q17, Q2, Q21, Q22, Q23, Q25, Q4, Q5, Q6, Q8: renamed from Q?; footprint (none) -> Package_TO_SOT_SMD:SOT-23_Handsoldering
- R1, R13, R15, R18, R2, R22, R3, R4, R5, R7, R9: renamed from R?; footprint (none) -> Resistor_SMD:R_0201_0603Metric_Pad0.64x0.40mm_HandSolder
- TP1, TP3: renamed from TP?; footprint (none) -> TestPoint:TestPoint_Pad_D1.5mm
- U1, U3: renamed from U?; footprint (none) -> Package_TO_SOT_SMD:TSOT-23-6
- gave numbers to parts that had none: 1
Connections:
- net labels added: +3V3, led00, led10, led11, led_01
- wire segments 183 -> 210
- no-connect marks 15 -> 11
Other:
- moved on the sheet: C1, C2, C3, C4, C5, C6, C7, D1, J1, J2, J3, J4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

Commit message: start main board pcb
Parts:
- added J?: power, TerminalBlock_Phoenix:TerminalBlock_Phoenix_MKDS-1,5-2_1x02_P5.00mm_Horizontal, symbol Connector_Generic:Conn_01x02
Connections:
- wire segments 210 -> 212
Other:
- moved on the sheet: C1, C2, C4, C5, J1, L1, R1, R2, TP1, U1

Commit message: Main board pcb rev1 done and ordered
Parts:
- added D2: BZT52C5V1+, Diode_SMD:D_SOD-123, symbol Device:D_Zener_Small
- added F1, F2: MC36232, Fuse:Fuse_1812_4532Metric_Castellated, symbol Device:Fuse
- added H1, H2, H3, H4: MountingHole_Pad, MountingHole:MountingHole_3.2mm_M3_Pad_TopBottom, symbol Mechanical:MountingHole_Pad
- added JP1, JP2: SolderJumper_2_Open, Jumper:SolderJumper-2_P1.3mm_Open_TrianglePad1.0x1.5mm, symbol Jumper:SolderJumper_2_Open
- added Q26: CPH3350-TL-W, Package_TO_SOT_SMD:SOT-23_Handsoldering, symbol Device:Q_PMOS_GSD
- added R23: 10k, Resistor_SMD:R_0603_1608Metric_Pad0.98x0.95mm_HandSolder, symbol Device:R_Small
- R1, R10, R11, R12, R13, R14, R15, R16, R17, R18, R19, R2, R20, R21, R22, R3, R4, R5, R6, R7, R8, R9: footprint Resistor_SMD:R_0201_0603Metric_Pad0.64x0.40mm_HandSolder -> Resistor_SMD:R_0603_1608Metric_Pad0.98x0.95mm_HandSolder
- U2: footprint RPi_Pico:RPi_Pico_SMD_TH -> MCU_RaspberryPi_and_Boards:RPi_Pico_SMD_TH
- gave numbers to parts that had none: 1
Connections:
- net labels added: combined_vin, led01, matrix_led_data, vled_fb, vled_sw, vsys_fb, vsys_sw
- net labels removed: 3v3, led_01
- wire segments 212 -> 251
Other:
- note added: "voltage drop might add up from protection stuffs. \nMake it bypassable by bridges to be safe"
- moved on the sheet: C1, C2, C3, C4, C5, J1, J3, J4, J5, J8, L1, Q10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

Commit message: Fix error in schema
burned 4 regulatorsy
Parts:
- Q1, Q12, Q15, Q18, Q24, Q3, Q7: value SBC847AWT1G -> BC848CWT1G
- U1, U3: symbol good_things:AP62250 -> main_board-rescue:AP62250-good_things
- U2: symbol MCU_RaspberryPi_and_Boards:Pico -> main_board-rescue:Pico-MCU_RaspberryPi_and_Boards
Connections:
- net vin: no longer U1.5 (en), U3.5 (en)
- no-connect marks 11 -> 13
Changed lines of the file:
@@
 NoConn ~ 4200 7550
 $Comp
-L good_things:AP62250 U1
+L main_board-rescue:AP62250-good_things U1
 U 1 1 60F7EF7C
 P 4950 2000
@@
 P 6800 5550
 F 0 "Q1" H 7000 5450 50  0000 L CNN
-F 1 "SBC847AWT1G" V 7050 5550 50  0000 L CNN
+F 1 "BC848CWT1G" V 7050 5550 50  0000 L CNN
 F 2 "Package_TO_SOT_SMD:SOT-323_SC-70_Handsoldering" H 7000 5650 50  0001 C CNN
 F 3 "~" H 6800 5550 50  0001 C CNN
@@
 	8800 5300 8800 4400
 Connection ~ 8800 5300
-$Comp
-L Device:Q_NPN_BEC Q3
-U 1 1 611FBC76
-P 8100 5550
-F 0 "Q3" H 8300 5450 50  0000 L CNN
-F 1 "SBC847AWT1G" V 8350 5550 50  0000 L CNN
-F 2 "Package_TO_SOT_SMD:SOT-323_SC-70_Handsoldering" H 8300 5650 50  0001 C CNN
-F 3 "~" H 8100 5550 50  0001 C CNN
-	1    8100 5550
-	1    0    0    -1
-$EndComp
 Wire Wire Line
 	8200 5350 8200 5300
@@
 	10050 5300 10050 4400
 Connection ~ 10050 5300
-$Comp
-L Device:Q_NPN_BEC Q7
-U 1 1 6120E7AD
-P 9350 5550
-F 0 "Q7" H 9550 5450 50  0000 L CNN
-F 1 "SBC847AWT1G" V 9600 5550 50  0000 L CNN
-F 2 "Package_TO_SOT_SMD:SOT-323_SC-70_Handsoldering" H 9550 5650 50  0001 C CNN
-F 3 "~" H 9350 5550 50  0001 C CNN
-	1    9350 5550
-	1    0    0    -1
-$EndComp
 Wire Wire Line
 	9450 5350 9450 5300
@@
 	11350 5300 11350 4400
 Connection ~ 11350 5300
-$Comp
-L Device:Q_NPN_BEC Q12
-U 1 1 612134FF
-P 10650 5550
-F 0 "Q12" H 10850 5450 50  0000 L CNN
-F 1 "SBC847AWT1G" V 10900 5550 50  0000 L CNN
-F 2 "Package_TO_SOT_SMD:SOT-323_SC-70_Handsoldering" H 10850 5650 50  0001 C CNN
-F 3 "~" H 10650 5550 50  0001 C CNN
-	1    10650 5550
-	1    0    0    -1
-$EndComp
 Wire Wire Line
 	10750 5350 10750 5300
@@
 	12650 5300 12650 4400
 Connection ~ 12650 5300
-$Comp
-L Device:Q_NPN_BEC Q15
-U 1 1 612181C0
-P 11950 5550
-F 0 "Q15" H 12150 5450 50  0000 L CNN
-F 1 "SBC847AWT1G" V 12200 5550 50  0000 L CNN
-F 2 "Package_TO_SOT_SMD:SOT-323_SC-70_Handsoldering" H 12150 5650 50  0001 C CNN
-F 3 "~" H 11950 5550 50  0001 C CNN
-	1    11950 5550
-	1    0    0    -1
-$EndComp
 Wire Wire Line
 	12050 5350 12050 5300
@@
 	14000 5300 14000 4400
 Connection ~ 14000 5300
-$Comp
-L Device:Q_NPN_BEC Q18
-U 1 1 6121D191
-P 13300 5550
-F 0 "Q18" H 13500 5450 50  0000 L CNN
-F 1 "SBC847AWT1G" V 13550 5550 50  0000 L CNN
-F 2 "Package_TO_SOT_SMD:SOT-323_SC-70_Handsoldering" H 13500 5650 50  0001 C CNN
-F 3 "~" H 13300 5550 50  0001 C CNN
-	1    13300 5550
-	1    0    0    -1
-$EndComp
 Wire Wire Line
 	13400 5350 13400 5300
@@
 	15350 5300 15350 4400
 Connection ~ 15350 5300
-$Comp
-L Device:Q_NPN_BEC Q24
-U 1 1 6122EEF6
-P 14650 5550
-F 0 "Q24" H 14850 5450 50  0000 L CNN
-F 1 "SBC847AWT1G" V 14900 5550 50  0000 L CNN
-F 2 "Package_TO_SOT_SMD:SOT-323_SC-70_Handsoldering" H 14850 5650 50  0001 C CNN
-F 3 "~" H 14650 5550 50  0001 C CNN
-	1    14650 5550
-	1    0    0    -1
-$EndComp
 Wire Wire Line
 	14750 5350 14750 5300
@@
 	4350 1600 4350 1850
 Connection ~ 4350 1850
-Wire Wire Line
-	4350 1850 4550 1850
 Connection ~ 3550 1850
 $Comp
@@
 	4050 1850 4350 1850
 Wire Wire Line
-	4550 1850 4550 1950
-Wire Wire Line
-	4550 1950 4650 1950
-Connection ~ 4550 1850
-Wire Wire Line
-	4550 1850 4650 1850
-Wire Wire Line
 	5250 1850 5250 1750
 Wire Wire Line
@@
 	6150 4650 6150 4700
 $Comp
-L good_things:AP62250 U3
+L main_board-rescue:AP62250-good_things U3
 U 1 1 61701BAD
 P 4750 4450
@@
 	4400 4500 4450 4500
 Wire Wire Line
-	4350 4300 4350 4400
-Wire Wire Line
-	4350 4400 4450 4400
-Wire Wire Line
-	4350 4300 4450 4300
-Wire Wire Line
 	5050 4300 5050 4200
 Wire Wire Line
@@
 	3700 4300 3800 4300
 Connection ~ 3800 4300
-Wire Wire Line
-	3800 4300 4350 4300
-Connection ~ 4350 4300
 Wire Wire Line
 	5250 4400 5850 4400
@@
 	4300 8850 4200 8850
 $Comp
-L MCU_RaspberryPi_and_Boards:Pico U2
+L main_board-rescue:Pico-MCU_RaspberryPi_and_Boards U2
 U 1 1 60F4C6D0
 P 3500 8500
@@
 Text Label 4300 8650 0    50   ~ 0
 matrix_led_data
+$Comp
+L Device:Q_NPN_BEC Q3
+U 1 1 61288A62
+P 8100 5550
+F 0 "Q3" H 8300 5450 50  0000 L CNN
+F 1 "BC848CWT1G" V 8350 5550 50  0000 L CNN
+F 2 "Package_TO_SOT_SMD:SOT-323_SC-70_Handsoldering" H 8300 5650 50  0001 C CNN
+F 3 "~" H 8100 5550 50  0001 C CNN
+	1    8100 5550
+	1    0    0    -1
+$EndComp
+$Comp
+L Device:Q_NPN_BEC Q7
+U 1 1 61289031
+P 9350 5550
+F 0 "Q7" H 9550 5450 50  0000 L CNN
+F 1 "BC848CWT1G" V 9600 5550 50  0000 L CNN
+F 2 "Package_TO_SOT_SMD:SOT-323_SC-70_Handsoldering" H 9550 5650 50  0001 C CNN
+F 3 "~" H 9350 5550 50  0001 C CNN
+	1    9350 5550
+	1    0    0    -1
+$EndComp
+$Comp
+L Device:Q_NPN_BEC Q12
+U 1 1 612896A8
+P 10650 5550
+F 0 "Q12" H 10850 5450 50  0000 L CNN
+F 1 "BC848CWT1G" V 10900 5550 50  0000 L CNN
+F 2 "Package_TO_SOT_SMD:SOT-323_SC-70_Handsoldering" H 10850 5650 50  0001 C CNN
+F 3 "~" H 10650 5550 50  0001 C CNN
+	1    10650 5550
+	1    0    0    -1
+$EndComp
+$Comp
+L Device:Q_NPN_BEC Q15
+U 1 1 6128998B
+P 11950 5550
+F 0 "Q15" H 12150 5450 50  0000 L CNN
+F 1 "BC848CWT1G" V 12200 5550 50  0000 L CNN
+F 2 "Package_TO_SOT_SMD:SOT-323_SC-70_Handsoldering" H 12150 5650 50  0001 C CNN
+F 3 "~" H 11950 5550 50  0001 C CNN
+	1    11950 5550
+	1    0    0    -1
+$EndComp
+$Comp
+L Device:Q_NPN_BEC Q18
+U 1 1 61289E8E
+P 13300 5550
+F 0 "Q18" H 13500 5450 50  0000 L CNN
+F 1 "BC848CWT1G" V 13550 5550 50  0000 L CNN
+F 2 "Package_TO_SOT_SMD:SOT-323_SC-70_Handsoldering" H 13500 5650 50  0001 C CNN
+F 3 "~" H 13300 5550 50  0001 C CNN
+	1    13300 5550
+	1    0    0    -1
+$EndComp
+$Comp
+L Device:Q_NPN_BEC Q24
+U 1 1 6128A14D
+P 14650 5550
+F 0 "Q24" H 14850 5450 50  0000 L CNN
+F 1 "BC848CWT1G" V 14900 5550 50  0000 L CNN
+F 2 "Package_TO_SOT_SMD:SOT-323_SC-70_Handsoldering" H 14850 5650 50  0001 C CNN
+F 3 "~" H 14650 5550 50  0001 C CNN
+	1    14650 5550
+	1    0    0    -1
+$EndComp
+Wire Wire Line
+	3800 4300 4450 4300
+NoConn ~ 4450 4400
+Wire Wire Line
+	4350 1850 4650 1850
+NoConn ~ 4650 1950
 $EndSCHEMATC

Commit message: Controller code and update pmos
Parts:
- Q13, Q17, Q2, Q22, Q25, Q5, Q8: value SI2365EDS-T1-GE3 -> CPH3350-TL-W
Changed lines of the file:
@@
 P 7400 5550
 F 0 "Q2" H 7605 5504 50  0000 L CNN
-F 1 "SI2365EDS-T1-GE3" V 7605 5595 50  0000 L CNN
+F 1 "CPH3350-TL-W" V 7605 5595 50  0000 L CNN
 F 2 "Package_TO_SOT_SMD:SOT-23_Handsoldering" H 7600 5650 50  0001 C CNN
 F 3 "~" H 7400 5550 50  0001 C CNN
@@
 P 8700 5550
 F 0 "Q5" H 8905 5504 50  0000 L CNN
-F 1 "SI2365EDS-T1-GE3" V 8905 5595 50  0000 L CNN
+F 1 "CPH3350-TL-W" V 8905 5595 50  0000 L CNN
 F 2 "Package_TO_SOT_SMD:SOT-23_Handsoldering" H 8900 5650 50  0001 C CNN
 F 3 "~" H 8700 5550 50  0001 C CNN
@@
 P 9950 5550
 F 0 "Q8" H 10155 5504 50  0000 L CNN
-F 1 "SI2365EDS-T1-GE3" V 10155 5595 50  0000 L CNN
+F 1 "CPH3350-TL-W" V 10155 5595 50  0000 L CNN
 F 2 "Package_TO_SOT_SMD:SOT-23_Handsoldering" H 10150 5650 50  0001 C CNN
 F 3 "~" H 9950 5550 50  0001 C CNN
@@
 P 11250 5550
 F 0 "Q13" H 11455 5504 50  0000 L CNN
-F 1 "SI2365EDS-T1-GE3" V 11455 5595 50  0000 L CNN
+F 1 "CPH3350-TL-W" V 11455 5595 50  0000 L CNN
 F 2 "Package_TO_SOT_SMD:SOT-23_Handsoldering" H 11450 5650 50  0001 C CNN
 F 3 "~" H 11250 5550 50  0001 C CNN
@@
 P 12550 5550
 F 0 "Q17" H 12755 5504 50  0000 L CNN
-F 1 "SI2365EDS-T1-GE3" V 12755 5595 50  0000 L CNN
+F 1 "CPH3350-TL-W" V 12755 5595 50  0000 L CNN
 F 2 "Package_TO_SOT_SMD:SOT-23_Handsoldering" H 12750 5650 50  0001 C CNN
 F 3 "~" H 12550 5550 50  0001 C CNN
@@
 P 13900 5550
 F 0 "Q22" H 14105 5504 50  0000 L CNN
-F 1 "SI2365EDS-T1-GE3" V 14105 5595 50  0000 L CNN
+F 1 "CPH3350-TL-W" V 14105 5595 50  0000 L CNN
 F 2 "Package_TO_SOT_SMD:SOT-23_Handsoldering" H 14100 5650 50  0001 C CNN
 F 3 "~" H 13900 5550 50  0001 C CNN
@@
 P 15250 5550
 F 0 "Q25" H 15455 5504 50  0000 L CNN
-F 1 "SI2365EDS-T1-GE3" V 15455 5595 50  0000 L CNN
+F 1 "CPH3350-TL-W" V 15455 5595 50  0000 L CNN
 F 2 "Package_TO_SOT_SMD:SOT-23_Handsoldering" H 15450 5650 50  0001 C CNN
 F 3 "~" H 15250 5550 50  0001 C CNN

Commit message: refactoring and segment
Parts:
- removed Q1, Q12, Q15, Q18, Q24, Q3, Q7: BC848CWT1G, Package_TO_SOT_SMD:SOT-323_SC-70_Handsoldering, symbol Device:Q_NPN_BEC
- added Q1, Q12, Q15, Q18, Q24, Q3, Q7: MCH3481-TL-W, Package_TO_SOT_SMD:SOT-323_SC-70_Handsoldering, symbol Device:Q_NMOS_GSD
Connections:
- net GND: now also Q1.2 (S), Q12.2 (S), Q15.2 (S), Q18.2 (S), Q24.2 (S), Q3.2 (S), Q7.2 (S)
- net a: now also Q1.1 (G)
- net b: now also Q3.1 (G)
- net c: now also Q7.1 (G)
- net d: now also Q12.1 (G)
- net e: now also Q15.1 (G)
- net f: now also Q18.1 (G)
- net g: now also Q24.1 (G)
- net at Q2.1 (G), R5.1: now also Q1.3 (D)
- net at Q5.1 (G), R7.1: now also Q3.3 (D)
- net at Q8.1 (G), R9.1: now also Q7.3 (D)
- net at Q13.1 (G), R13.1: now also Q12.3 (D)
- net at Q17.1 (G), R15.1: now also Q15.3 (D)
- net at Q22.1 (G), R18.1: now also Q18.3 (D)
- net at Q25.1 (G), R22.1: now also Q24.3 (D)
